Commit message: Add URDF and launch files for Odometry FIle robot
- Created display.launch for visualizing the robot in RViz.
- Created gazebo.launch for simulating the robot in Gazebo.
- Added package.xml for Odometry FIle with necessary dependencies.
- Included Odometry FIle.csv for robot component specifications.
- Added Odometry FIle.urdf for the robot's URDF description.
- Updated ct.urdf to reflect changes in link and joint names for consistency.

File: ros/src/ct_description/asd/urdf/urdf/Odometry FIle.urdf (robot description, URDF)
Before this commit: robot ct, 6 links, 5 joints
Links:
- removed link taitc_lidar_link
- added link Lidar, mass 0.0962112750161875; collision mesh filename=package://Odometry FIle/meshes/Lidar.STL; visual mesh filename=package://Odometry FIle/meshes/Lidar.STL
Joints:
- removed joint taitc_lidar_link
- added joint Lidar: type continuous, parent base_link, child Lidar, origin xyz=0.708399374631133 -1.37350613548206 0.854171401767211 rpy=1.5707963267949 0 1.90864148584851, axis 0 1 0
