Commit message: teleop + encoder + launch

File: ros/src/ct_description/urdf/ct.urdf (robot description, URDF)
Before this commit: robot cyber_truck, 3 links, 2 joints
Links:
- removed link base_footprint
- removed link lidar_link
- link base_link: mass None -> 5.0; geometry collision box size=0.5 0.3 0.1; visual box size=0.5 0.3 0.1
Joints:
- removed joint base_footprint_joint
- removed joint lidar_joint

Commit message: Add LIDAR link and joint to URDF; update launch file for teleop node

File: ros/src/ct_description/urdf/ct.urdf (robot description, URDF)
Before this commit: robot my_diffdrive_robot, 1 links, 0 joints
Links:
- added link taitc_lidar_link, mass 5.0; collision cylinder length=0.05 radius=0.03; visual cylinder length=0.05 radius=0.03
Joints:
- added joint lidar_joint: type fixed, parent base_link, child taitc_lidar_link, origin xyz=0.1 0 0.1 rpy=0 0 0

Commit message: fix: correct serial comment and add URDF and CSV files for robot description

File: ros/src/ct_description/urdf/ct.urdf (robot description, URDF)
Before this commit: robot my_diffdrive_robot, 2 links, 1 joints
Links:
- removed link taitc_lidar_link
- added link Lidar, mass 0.0962112750161875; collision mesh filename=package://Odometry FIle/meshes/Lidar.STL; visual mesh filename=package://Odometry FIle/meshes/Lidar.STL
- added link Wheel1, mass 0.224922326033761; collision mesh filename=package://Odometry FIle/meshes/Wheel1.STL; visual mesh filename=package://Odometry FIle/meshes/Wheel1.STL
- added link Wheel2, mass 0.224922326033761; collision mesh filename=package://Odometry FIle/meshes/Wheel2.STL; visual mesh filename=package://Odometry FIle/meshes/Wheel2.STL
- added link Wheel3, mass 0.224922326033761; collision mesh filename=package://Odometry FIle/meshes/Wheel3.STL; visual mesh filename=package://Odometry FIle/meshes/Wheel3.STL
- added link Wheel4, mass 0.224922326033761; collision mesh filename=package://Odometry FIle/meshes/Wheel4.STL; visual mesh filename=package://Odometry FIle/meshes/Wheel4.STL
- link base_link: mass 5.0 -> 0.249821153529968; geometry collision mesh filename=package://Odometry FIle/meshes/base_link.STL; visual mesh filename=package://Odometry FIle/meshes/base_link.STL
Joints:
- removed joint lidar_joint
- added joint Lidar: type continuous, parent base_link, child Lidar, origin xyz=0.708399374631133 -1.37350613548206 0.854171401767211 rpy=1.5707963267949 0 1.90864148584851, axis 0 1 0
- added joint Wheel1: type continuous, parent base_link, child Wheel1, origin xyz=0.56391 -1.444 0.99365 rpy=1.5708 0.013855 0, axis 0 0 1
- added joint Wheel2: type continuous, parent base_link, child Wheel2, origin xyz=0.56391 -1.259 0.99365 rpy=-1.5708 0.38576 -3.1416, axis 0 0 1
- added joint Wheel3: type continuous, parent base_link, child Wheel3, origin xyz=0.88391 -1.444 0.99365 rpy=1.5708 -0.17346 0, axis 0 0 1
- added joint Wheel4: type continuous, parent base_link, child Wheel4, origin xyz=0.88391 -1.259 0.99365 rpy=1.5708 -0.073815 0, axis 0 0 1

Commit message: fix: update taitc_lidar_joint to be fixed and improve structure

File: ros/src/ct_description/urdf/ct.urdf (robot description, URDF)
Before this commit: robot ct, 6 links, 5 joints
Joints:
- removed joint taitc_lidar_link
- added joint taitc_lidar_joint: type fixed, parent base_link, child taitc_lidar_link, origin xyz=0.708399374631133 -1.37350613548206 0.854171401767211 rpy=1.5707963267949 0 1.90864148584851

Commit message: fix: correct rpy values for taitc_lidar_joint in URDF

File: ros/src/ct_description/urdf/ct.urdf (robot description, URDF)
Before this commit: robot ct, 6 links, 5 joints
Joints:
- joint taitc_lidar_joint: origin xyz=0.708399374631133 -1.37350613548206 0.854171401767211 rpy=1.5707963267949 0 1.90864148584851 -> xyz=0.708399374631133 -1.37350613548206 0.854171401767211 rpy=0 0 0

Commit message: refactor: clean up URDF structure and align wheel names with ros2_control

File: ros/src/ct_description/urdf/ct.urdf (robot description, URDF)
Before this commit: robot ct, 6 links, 5 joints
Links:
- removed link Wheel1
- removed link Wheel2
- removed link Wheel3
- removed link Wheel4
- added link front_left_wheel_link, mass 0.224922326033761; collision mesh filename=package://Odometry FIle/meshes/Wheel1.STL; visual mesh filename=package://Odometry FIle/meshes/Wheel1.STL
- added link front_right_wheel_link, mass 0.224922326033761; collision mesh filename=package://Odometry FIle/meshes/Wheel2.STL; visual mesh filename=package://Odometry FIle/meshes/Wheel2.STL
- added link rear_left_wheel_link, mass 0.224922326033761; collision mesh filename=package://Odometry FIle/meshes/Wheel3.STL; visual mesh filename=package://Odometry FIle/meshes/Wheel3.STL
- added link rear_right_wheel_link, mass 0.224922326033761; collision mesh filename=package://Odometry FIle/meshes/Wheel4.STL; visual mesh filename=package://Odometry FIle/meshes/Wheel4.STL
Joints:
- removed joint Wheel1
- removed joint Wheel2
- removed joint Wheel3
- removed joint Wheel4
- added joint front_left_wheel_joint: type continuous, parent base_link, child front_left_wheel_link, origin xyz=0.56391 -1.444 0.99365 rpy=1.5708 0.013855 0, axis 0 0 1
- added joint front_right_wheel_joint: type continuous, parent base_link, child front_right_wheel_link, origin xyz=0.56391 -1.259 0.99365 rpy=-1.5708 0.38576 -3.1416, axis 0 0 1
- added joint rear_left_wheel_joint: type continuous, parent base_link, child rear_left_wheel_link, origin xyz=0.88391 -1.444 0.99365 rpy=1.5708 -0.17346 0, axis 0 0 1
- added joint rear_right_wheel_joint: type continuous, parent base_link, child rear_right_wheel_link, origin xyz=0.88391 -1.259 0.99365 rpy=1.5708 -0.073815 0, axis 0 0 1

Commit message: refactor: clean up URDF structure and align wheel names with ros2_control

File: ros/src/ct_description/urdf/ct.urdf (robot description, URDF)
Before this commit: robot ct, 6 links, 5 joints
Links:
- removed link front_left_wheel_link
- removed link front_right_wheel_link
- removed link rear_left_wheel_link
- removed link rear_right_wheel_link
- added link dummy_root_link
- link base_link: mass 0.249821153529968 -> 0.5
- link taitc_lidar_link: mass 0.0962112750161875 -> None; geometry visual mesh filename=package://Odometry FIle/meshes/taitc_lidar_link.STL
Joints:
- removed joint front_left_wheel_joint
- removed joint front_right_wheel_joint
- removed joint rear_left_wheel_joint
- removed joint rear_right_wheel_joint
- added joint base_joint: type fixed, parent dummy_root_link, child base_link, origin xyz=0 0 0 rpy=0 0 0
- joint taitc_lidar_joint: origin xyz=0.708399374631133 -1.37350613548206 0.854171401767211 rpy=0 0 0 -> xyz=0.708 -1.3735 0.854 rpy=0 0 0

Commit message: Changes to be committed:

File: ros/src/ct_description/urdf/ct.urdf (robot description, URDF)
Before this commit: robot ct, 3 links, 2 joints
Links:
- removed link dummy_root_link
Joints:
- added joint base_footprint_to_base_link: type fixed, parent base_footprint, child base_link, origin xyz=0 0 0 rpy=0 0 0
- joint base_joint: parent dummy_root_link -> (none)

Commit message: refactor: update URDF structure and enhance wheel definitions for improved clarity

File: ros/src/ct_description/urdf/ct.urdf (robot description, URDF)
Before this commit: robot ct, 2 links, 3 joints
Links:
- added link Wheel1, mass 0.224922326033761; collision mesh filename=package://Odometry FIle/meshes/Wheel1.STL; visual mesh filename=package://Odometry FIle/meshes/Wheel1.STL
- added link left_front_wheel_names, mass 0.224922326033761; collision mesh filename=package://Odometry FIle/meshes/left_front_wheel_names.STL; visual mesh filename=package://Odometry FIle/meshes/left_front_wheel_names.STL
- added link left_rear_wheel_names, mass 0.224922326033761; collision mesh filename=package://Odometry FIle/meshes/left_rear_wheel_names.STL; visual mesh filename=package://Odometry FIle/meshes/left_rear_wheel_names.STL
- added link right_front_wheel_names, mass 0.224922326033761; collision mesh filename=package://Odometry FIle/meshes/right_front_wheel_names.STL; visual mesh filename=package://Odometry FIle/meshes/right_front_wheel_names.STL
- link base_link: mass 0.5 -> 0.249821153529968
- link taitc_lidar_link: mass None -> 0.0962112750161875; geometry collision mesh filename=package://Odometry FIle/meshes/taitc_lidar_link.STL; visual mesh filename=package://Odometry FIle/meshes/taitc_lidar_link.STL
Joints:
- removed joint base_footprint_to_base_link
- removed joint base_joint
- removed joint taitc_lidar_joint
- added joint left_front_wheel_names: type continuous, parent base_link, child left_front_wheel_names, origin xyz=0.88391 -1.259 0.99365 rpy=1.5708 -0.073815 0, axis 0 0 1
- added joint left_rear_wheel_names: type continuous, parent base_link, child left_rear_wheel_names, origin xyz=0.56391 -1.259 0.99365 rpy=-1.5708 0.38576 -3.1416, axis 0 0 1
- added joint right_front_wheel_names: type continuous, parent base_link, child right_front_wheel_names, origin xyz=0.88391 -1.444 0.99365 rpy=1.5708 -0.17346 0, axis 0 0 1
- added joint right_rear_wheel_names: type continuous, parent base_link, child right_rear_wheel_names, origin xyz=0.56391 -1.444 0.99365 rpy=1.5708 0.013855 0, axis 0 0 1
- added joint taitc_lidar_link: type continuous, parent base_link, child taitc_lidar_link, origin xyz=0.708399374631133 -1.37350613548206 0.854171401767211 rpy=1.5707963267949 0 1.90864148584851, axis 0 1 0

Commit message: feat: implement motion controller and odometry nodes; update launch configuration

File: ros/src/ct_description/urdf/ct.urdf (robot description, URDF)
Before this commit: robot Odometry FIle, 6 links, 5 joints
Links:
- removed link Wheel1
- removed link left_front_wheel_names
- removed link left_rear_wheel_names
- removed link right_front_wheel_names
- added link left_front_wheel
- added link left_rear_wheel
- added link right_front_wheel
- added link right_rear_wheel
- link taitc_lidar_link: mass 0.0962112750161875 -> None; geometry 
Joints:
- removed joint left_front_wheel_names
- removed joint left_rear_wheel_names
- removed joint right_front_wheel_names
- removed joint right_rear_wheel_names
- removed joint taitc_lidar_link
- added joint left_front_wheel_joint: type continuous, parent base_link, child left_front_wheel, origin xyz=0.88391 -1.259 0.99365 rpy=1.5708 -0.073815 0, axis 0 0 1
- added joint left_rear_wheel_joint: type continuous, parent base_link, child left_rear_wheel, origin xyz=0.56391 -1.259 0.99365 rpy=-1.5708 0.38576 -3.1416, axis 0 0 1
- added joint right_front_wheel_joint: type continuous, parent base_link, child right_front_wheel, origin xyz=0.88391 -1.444 0.99365 rpy=1.5708 -0.17346 0, axis 0 0 1
- added joint right_rear_wheel_joint: type continuous, parent base_link, child right_rear_wheel, origin xyz=0.56391 -1.444 0.99365 rpy=1.5708 0.013855 0, axis 0 0 1
- added joint taitc_lidar_joint: type continuous, parent base_link, child taitc_lidar_link, origin xyz=0.708399374631133 -1.37350613548206 0.854171401767211 rpy=1.5707963267949 0 1.90864148584851, axis 0 1 0

Commit message: feat: add base footprint link and joint; update LiDAR joint type to fixed

File: ros/src/ct_description/urdf/ct.urdf (robot description, URDF)
Before this commit: robot Odometry_File, 6 links, 5 joints
Links:
- added link base_footprint
Joints:
- added joint base_footprint_joint: type fixed, parent base_footprint, child base_link, origin xyz=0 0 0 rpy=0 0 0
- joint taitc_lidar_joint: type continuous -> fixed

Commit message: Add ros2_joy_twist package for joystick to Twist mapping
- Implemented the `ros2_joy_twist` package to convert joystick inputs to Twist messages for robot control.
- Created `joy_to_twist.py` to handle joystick input and publish corresponding Twist commands.
- Added launch files for testing with turtlesim and standalone joystick node.
- Included parameter mapping in `mappings.yaml` for customizable joystick configuration.
- Defined package metadata in `package.xml` and `setup.py`.
- Added necessary dependencies for ROS 2 and included setup configuration.

File: ros/src/ct_description/urdf/ct.urdf (robot description, URDF)
Before this commit: robot Odometry_File, 7 links, 6 joints
Links:
- removed link taitc_lidar_link
- added link lidar_link
Joints:
- removed joint taitc_lidar_joint
- added joint lidar_joint: type fixed, parent base_link, child lidar_link, origin xyz=0.708399374631133 -1.37350613548206 0.854171401767211 rpy=1.5707963267949 0 1.90864148584851, axis 0 1 0

Commit message: Refactor lidar_joint origin and axis parameters for consistency

File: ros/src/ct_description/urdf/ct.urdf (robot description, URDF)
Before this commit: robot Odometry_File, 7 links, 6 joints
Joints:
- joint lidar_joint: axis 0 1 0 -> (none); origin xyz=0.708399374631133 -1.37350613548206 0.854171401767211 rpy=1.5707963267949 0 1.90864148584851 -> xyz=0.708  -1.374  0.854 rpy=0 0 0

Commit message: ct urdf

File: ros/src/ct_description/urdf/ct.urdf (robot description, URDF)
Before this commit: robot Odometry_File, 7 links, 6 joints
Joints:
- joint lidar_joint: origin xyz=0.708  -1.374  0.854 rpy=0 0 0 -> xyz=0.708  -1.374  1.2 rpy=0 0 0

Commit message: Refactor URDF for base link and wheel joints; update positions and remove comments

File: ros/src/ct_description/urdf/ct.urdf (robot description, URDF)
Before this commit: robot Odometry_File, 7 links, 6 joints
Joints:
- joint base_footprint_joint: origin xyz=0 0 0 rpy=0 0 0 -> xyz=0 0 0.1 rpy=0 0 0
- joint left_front_wheel_joint: origin xyz=0.88391 -1.259 0.99365 rpy=1.5708 -0.073815 0 -> xyz=0.165 0.105 0.1 rpy=-1.5708 0 0
- joint left_rear_wheel_joint: origin xyz=0.56391 -1.259 0.99365 rpy=-1.5708 0.38576 -3.1416 -> xyz=-0.165 0.105 0.1 rpy=-1.5708 0 0
- joint lidar_joint: origin xyz=0.708  -1.374  1.2 rpy=0 0 0 -> xyz=0 0 0.2 rpy=0 0 0
- joint right_front_wheel_joint: origin xyz=0.88391 -1.444 0.99365 rpy=1.5708 -0.17346 0 -> xyz=0.165 -0.105 0.1 rpy=-1.5708 0 0
- joint right_rear_wheel_joint: origin xyz=0.56391 -1.444 0.99365 rpy=1.5708 0.013855 0 -> xyz=-0.165 -0.105 0.1 rpy=-1.5708 0 0

Commit message: Update URDF for cybetruck: adjust base link position, add visual geometry for wheels, and refine joint origins

File: ros/src/ct_description/urdf/ct.urdf (robot description, URDF)
Before this commit: robot Odometry_File, 7 links, 6 joints
Links:
- link left_front_wheel: geometry visual cylinder length=0.04 radius=0.2
- link left_rear_wheel: geometry visual cylinder length=0.04 radius=0.2
- link right_front_wheel: geometry visual cylinder length=0.04 radius=0.2
- link right_rear_wheel: geometry visual cylinder length=0.04 radius=0.2
Joints:
- joint base_footprint_joint: origin xyz=0 0 0.1 rpy=0 0 0 -> xyz=0 0 0.2 rpy=0 0 0
- joint left_front_wheel_joint: origin xyz=0.165 0.105 0.1 rpy=-1.5708 0 0 -> xyz=0.165 0.14 0.2 rpy=-1.5708 0 0
- joint left_rear_wheel_joint: origin xyz=-0.165 0.105 0.1 rpy=-1.5708 0 0 -> xyz=-0.165 0.14 0.2 rpy=-1.5708 0 0
- joint right_front_wheel_joint: origin xyz=0.165 -0.105 0.1 rpy=-1.5708 0 0 -> xyz=0.165 -0.14 0.2 rpy=-1.5708 0 0
- joint right_rear_wheel_joint: origin xyz=-0.165 -0.105 0.1 rpy=-1.5708 0 0 -> xyz=-0.165 -0.14 0.2 rpy=-1.5708 0 0

Commit message: 13

File: ros/src/ct_description/urdf/ct.urdf (robot description, URDF)
Before this commit: robot cybetruck, 7 links, 6 joints
Links:
- link left_front_wheel: geometry visual cylinder length=0.04 radius=0.1
- link left_rear_wheel: geometry visual cylinder length=0.04 radius=0.1
- link right_front_wheel: geometry visual cylinder length=0.04 radius=0.1
- link right_rear_wheel: geometry visual cylinder length=0.04 radius=0.1
Joints:
- joint base_footprint_joint: origin xyz=0 0 0.2 rpy=0 0 0 -> xyz=0 0 0.1 rpy=0 0 0
- joint left_front_wheel_joint: origin xyz=0.165 0.14 0.2 rpy=-1.5708 0 0 -> xyz=0.165 0.105 0.1 rpy=-1.5708 0 0
- joint left_rear_wheel_joint: origin xyz=-0.165 0.14 0.2 rpy=-1.5708 0 0 -> xyz=-0.165 0.105 0.1 rpy=-1.5708 0 0
- joint right_front_wheel_joint: origin xyz=0.165 -0.14 0.2 rpy=-1.5708 0 0 -> xyz=0.165 -0.105 0.1 rpy=-1.5708 0 0
- joint right_rear_wheel_joint: origin xyz=-0.165 -0.14 0.2 rpy=-1.5708 0 0 -> xyz=-0.165 -0.105 0.1 rpy=-1.5708 0 0

Commit message: Update lidar joint orientation in URDF to correct rotation

File: ros/src/ct_description/urdf/ct.urdf (robot description, URDF)
Before this commit: robot Odometry_File, 7 links, 6 joints
Joints:
- joint lidar_joint: origin xyz=0 0 0.2 rpy=0 0 0 -> xyz=0 0 0.2 rpy=0 0 3.14

Commit message: bsae_footprint to base link

File: ros/src/ct_description/urdf/ct.urdf (robot description, URDF)
Before this commit: robot Odometry_File, 7 links, 6 joints
Links:
- removed link base_footprint
- link base_link: mass 0.249821153529968 -> None; geometry 
Joints:
- removed joint base_footprint_joint
- added joint base_link_joint: type fixed, parent base_link, child base_link, origin xyz=0 0 0.1 rpy=0 0 0

Commit message: Revert "bsae_footprint to base link"
This reverts commit 30269300e62e0fae1fd32a26697bd6a463c5e692.

File: ros/src/ct_description/urdf/ct.urdf (robot description, URDF)
Before this commit: robot Odometry_File, 6 links, 6 joints
Links:
- added link base_footprint
- link base_link: mass None -> 0.249821153529968; geometry collision mesh filename=package://Odometry FIle/meshes/base_link.STL; visual mesh filename=package://Odometry FIle/meshes/base_link.STL
Joints:
- removed joint base_link_joint
- added joint base_footprint_joint: type fixed, parent base_footprint, child base_link, origin xyz=0 0 0.1 rpy=0 0 0
